File: D-class.brd (EAGLE design)
At the start: 65 parts, among them IC1 TPA3118D2, IC2 78L12, IC3 7812

Commit message: 後はシルクのみ
Parts:
- added C22, C29, C30, C33: 100p, my_rcl:1608
- added HOLE1, HOLE2, HOLE3, HOLE4: HOLE_3.2, Document_Robotech:HOLE_3.2
- C11, C23: device my_rcl:E2,5-8 -> my_rcl:E5-10
- moved C23 24.7 mm to (48.3, 7.62)
- moved C12 24.1 mm to (17.8, 18.7)
- moved IC2 23.6 mm to (19.7, 14.9)
- moved JP1 23.4 mm to (2.54, 12.7)
- moved JP3 23.4 mm to (2.54, 33.0)
- moved C13 23.4 mm to (18.7, 8.57)
- moved C1 23.1 mm to (16.5, 37.8)
- moved C10 23.1 mm to (27.9, 32.7)
- moved C14 23.1 mm to (42.5, 36.5)
- moved C2 23.1 mm to (16.5, 34.6)
- moved C20 23.1 mm to (40.0, 25.1)
- moved C25 23.1 mm to (40.0, 22.5)
- moved C3 23.1 mm to (16.5, 31.4)
- moved C31 23.1 mm to (56.5, 47.9)
- moved C4 23.1 mm to (16.5, 28.3)
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Connections:
- net GND: now also C22.2, C29.2, C30.2, C33.2
- net N$25: now also C29.1
- net N$26: now also C22.1
- net N$27: now also C30.1
- net N$28: now also C33.1
Routing:
- net VCC: track 28.7 -> 31.3 mm
- net AVCC: track 88.0 -> 86.7 mm
- net SLEEP: track 35.2 -> 34.3 mm
- net N$27: track 55.3 -> 56.2 mm
- net N$25: track 58.9 -> 59.6 mm
Other:
- board outline added: 69.8 x 53 mm
- board text added: "D-CLASS AMP"
- board text added: "ver 1.0"

Commit message: できた
Parts:
- added C34: 100p, my_rcl:1608
- added FB1: FB-1608, my_rcl:1608
- C22: value 100p -> 1000u; device my_rcl:1608 -> my_rcl:E5-10
- C23: value 220u -> 0.1u; device my_rcl:E5-10 -> my_rcl:2012
- C25: value 0.1u -> 100u; device my_rcl:2012 -> my_rcl:E2.5-6.5
- C28: value 100u -> 0.47u; device my_rcl:E2.5-6.5 -> my_rcl:C050-030X075
- C29, C30: value 100p -> 0.47u; device my_rcl:1608 -> my_rcl:C050-030X075
- C32, C35: value 0.47u -> 100p; device my_rcl:C050-030X075 -> my_rcl:1608
- C36: value 0.47u -> 100u; device my_rcl:C050-030X075 -> my_rcl:E2.5-6.5
- moved C36 44.2 mm to (12.4, 19.1), turned to 180 degrees
- moved C23 34.8 mm to (40.6, 41.6)
- moved C28 29.9 mm to (56.5, 47.9)
- moved C26 29.1 mm to (47.6, 44.8), turned to 180 degrees
- moved C31 27.3 mm to (56.5, 20.6), turned to 0 degrees
- moved C27 25.4 mm to (47.6, 19.4)
- moved C22 23.1 mm to (48.3, 7.62), turned to 180 degrees
- moved C24 19.1 mm to (40.0, 22.5)
- moved C29 15.3 mm to (56.5, 16.2), turned to 0 degrees
- moved C30 11.5 mm to (56.5, 43.5), turned to 180 degrees
- moved C32 11.2 mm to (64.5, 24.1)
- moved C33 9.25 mm to (61.9, 30.5), turned to 90 degrees
- moved C35 8.95 mm to (64.5, 39.4), turned to 0 degrees
- moved C25 5.75 mm to (39.4, 16.8), turned to 90 degrees
- moved C12 3.19 mm to (18.1, 15.6), turned to 270 degrees
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Connections:
- new net N$7: C12.1, C36.+, FB1.2, IC2.3
- net AVCC: now also C25.+; no longer C26.+
- net GND: now also C22.-, C23.2, C25.-, C28.2, C29.1, C31.1, C32.2, C34.2, C36.-; no longer C22.2, C23.-, C25.2, C28.-, C29.2, C31.2, C32.1, C36.1
- net N$25: now also C31.2, C33.1; no longer C29.1, C36.2
- net N$26: now also C29.2, C32.1; no longer C22.1, C32.2
- net N$27: now also C34.1; no longer C35.1
- net N$28: now also C28.1, C35.1; no longer C31.1, C33.1
- net PVCC: now also C22.+, C23.1, C26.+; no longer C23.+, C25.1, C28.+
- net VCC: now also FB1.1; no longer C12.1, IC2.3
Routing:
- net N$7: track 0.00 -> 9.61 mm
- net N$27: track 56.2 -> 48.1 mm
- net N$25: track 59.6 -> 52.4 mm
- net VCC: track 31.3 -> 27.9 mm
- net AVCC: track 86.7 -> 84.8 mm
- net N$10: track 47.8 -> 49.3 mm
- net N$26: track 69.4 -> 68.9 mm
- net N$28: track 64.2 -> 63.6 mm
Other:
- board size 69.8 x 53 mm -> 69.8 x 53.3 mm
